Commit message: Rename to timmy2

File: timmy2_description/urdf/jimmy.urdf.xacro (robot description, xacro)
@@ -41,5 +41,5 @@
     </xacro:property>
     <!-- Import Gazebo-customization stuff -->
-    <xacro:include filename="$(find jimmy2_description)/urdf/test.gazebo" />
+    <xacro:include filename="$(find timmy2_description)/urdf/test.gazebo" />
     <link name="world" />
     <joint name="fixed" type="fixed">
@@ -58,5 +58,5 @@
             <xacro:insert_block name="torso_origin"/>
             <geometry>
-                <mesh filename="package://jimmy2_description/meshes/torso.dae"/>
+                <mesh filename="package://timmy2_description/meshes/torso.dae"/>
             </geometry>
             <material name="orange"/>
@@ -91,5 +91,5 @@
             <xacro:insert_block name="l_sho_pitch_block_origin"/>
             <geometry>
-                <mesh filename="package://jimmy2_description/meshes/l_sho_pitch.dae"/>
+                <mesh filename="package://timmy2_description/meshes/l_sho_pitch.dae"/>
             </geometry>
             <material name="black"/>
@@ -120,5 +120,5 @@
             <xacro:insert_block name="l_sho_pitch_bracket_origin"/>
             <geometry>
-                <mesh filename="package://jimmy2_description/meshes/l_sho_bracket.dae"/>
+                <mesh filename="package://timmy2_description/meshes/l_sho_bracket.dae"/>
             </geometry>
             <material name="black"/>
@@ -148,5 +148,5 @@
             <xacro:insert_block name="l_sho_roll_block_origin"/>
             <geometry>
-                <mesh filename="package://jimmy2_description/meshes/l_sho_roll.dae"/>
+                <mesh filename="package://timmy2_description/meshes/l_sho_roll.dae"/>
             </geometry>
             <material name="black"/>
@@ -180,5 +180,5 @@
             <origin xyz="0 0 0" rpy="0 0 0"/>
             <geometry>
-                <mesh filename="package://jimmy2_description/meshes/r_hand2.dae"/>
+                <mesh filename="package://timmy2_description/meshes/r_hand2.dae"/>
             </geometry>
             <material name="black"/>
@@ -200,5 +200,5 @@
             <origin xyz="0 0 0" rpy="0 0 0"/>
             <geometry>
-                <mesh filename="package://jimmy2_description/meshes/r_forearm2.dae"/>
+                <mesh filename="package://timmy2_description/meshes/r_forearm2.dae"/>
             </geometry>
             <material name="black"/>

File: timmy2_description/urdf/test.urdf.xacro (robot description, xacro)
@@ -29,5 +29,5 @@
     </xacro:property>
     <!-- Import Gazebo-customization stuff -->
-    <xacro:include filename="$(find jimmy2_description)/urdf/test.gazebo" />
+    <xacro:include filename="$(find timmy2_description)/urdf/test.gazebo" />
     <link name="world" />
     <joint name="fixed" type="fixed">

File: timmy2_description/urdf/timmy2.urdf.xacro (robot description, xacro)
@@ -1,4 +1,4 @@
 <?xml version="1.0"?>
-<robot name="jimmy2" xmlns:xacro="http://www.ros.org/wiki/xacro">
+<robot name="timmy2" xmlns:xacro="http://www.ros.org/wiki/xacro">
     <xacro:property name="mass" value="0.2" />
     <xacro:property name="bracket_mass" value="0.01" />
@@ -12,5 +12,5 @@
     <xacro:property name="height3" value="1" /> <!-- Link 3 -->
     <xacro:property name="base_height" value="1.0" />
-    <xacro:property name="package_name" value="jimmy2_description" />
+    <xacro:property name="package_name" value="timmy2_description" />
     <xacro:property name="mesh_dir" value="meshes2" />
     <xacro:property name="torso_origin">
@@ -149,5 +149,5 @@
     </xacro:property>
     <!-- Import Gazebo-customization stuff -->
-    <xacro:include filename="$(find jimmy2_description)/urdf/test.gazebo" />
+    <xacro:include filename="$(find timmy2_description)/urdf/test.gazebo" />
     <link name="world" />
     <joint name="base_fixed" type="fixed">
@@ -736,5 +736,5 @@
     <gazebo>
         <plugin name="gazebo_ros_control" filename="libgazebo_ros_control.so">
-            <robotNamespace>/jimmy2</robotNamespace><!-- important - namespace mustbe correct -->
+            <robotNamespace>/timmy2</robotNamespace><!-- important - namespace mustbe correct -->
         </plugin>
     </gazebo>
