Commit message: Add control to elbow twist joints. Renamed test.gazebo to timmy2.gazebo

File: timmy2_description/urdf/timmy2.urdf.xacro (robot description, xacro)
@@ -149,5 +149,5 @@
     </xacro:property>
     <!-- Import Gazebo-customization stuff -->
-    <xacro:include filename="$(find timmy2_description)/urdf/test.gazebo" />
+    <xacro:include filename="$(find timmy2_description)/urdf/timmy2.gazebo" />
     <link name="world" />
     <joint name="base_fixed" type="fixed">

File: timmy2_description/urdf/timmy3.urdf.xacro (robot description, xacro)
@@ -167,5 +167,5 @@
     </xacro:property>
     <!-- Import Gazebo-customization stuff -->
-    <xacro:include filename="$(find timmy2_description)/urdf/test.gazebo" />
+    <xacro:include filename="$(find timmy2_description)/urdf/timmy2.gazebo" />
     <link name="world" />
     <joint name="base_fixed" type="fixed">
@@ -791,4 +791,14 @@
         </actuator>
     </transmission>
+    <transmission name="left_elbow_twist_tran">
+        <type>transmission_interface/SimpleTransmission</type>
+        <joint name="left_elbow_twist">
+            <hardwareInterface>hardware_interface/EffortJointInterface</hardwareInterface>
+        </joint>
+        <actuator name="motor5b">
+            <hardwareInterface>hardware_interface/EffortJointInterface</hardwareInterface>
+            <mechanicalReduction>1</mechanicalReduction>
+        </actuator>
+    </transmission>
     <transmission name="right_elbow_tran">
         <type>transmission_interface/SimpleTransmission</type>
@@ -797,4 +807,14 @@
         </joint>
         <actuator name="motor6">
+            <hardwareInterface>hardware_interface/EffortJointInterface</hardwareInterface>
+            <mechanicalReduction>1</mechanicalReduction>
+        </actuator>
+    </transmission>
+    <transmission name="right_elbow_twist_tran">
+        <type>transmission_interface/SimpleTransmission</type>
+        <joint name="right_elbow_twist">
+            <hardwareInterface>hardware_interface/EffortJointInterface</hardwareInterface>
+        </joint>
+        <actuator name="motor6b">
             <hardwareInterface>hardware_interface/EffortJointInterface</hardwareInterface>
             <mechanicalReduction>1</mechanicalReduction>
